File: pcb/kicad/pcb.kicad_pcb (KiCad board)
At the start: 2 copper layers, 54.6 x 53.3 mm, 24 parts, among them J1 Raspberry_Pi_2_3, U1 MCP4822, U2 TL082, U3 TL082, U4 MOC3022M

Commit message: pcb, laser_screenshot
Parts:
- removed RLED1: 510R, Resistor_THT:R_Axial_DIN0207_L6.3mm_D2.5mm_P10.16mm_Horizontal
- removed U4: MOC3022M, Package_DIP:DIP-6_W7.62mm
- removed buttons1: Conn_01x04_Male, Connector_PinHeader_2.54mm:PinHeader_1x04_P2.54mm_Horizontal
- removed laser1: Conn_01x02_Male, Connector_PinHeader_2.54mm:PinHeader_1x02_P2.54mm_Horizontal
- added LCD1: Conn_01x04_Female, Connector_PinSocket_2.54mm:PinSocket_1x04_P2.54mm_Horizontal, F.Cu at (223.8, 37.2)
- added LCD_backligh1: Conn_01x02_Female, Connector_PinSocket_2.54mm:PinSocket_1x02_P2.54mm_Horizontal, F.Cu at (211.6, 37.2)
- added Q1: BC547, Package_TO_SOT_THT:TO-92_Inline, F.Cu at (252.7, 43.3)
- added Q2: BC547, Package_TO_SOT_THT:TO-92_Inline, F.Cu at (260.1, 43.3)
- added Q3: BC547, Package_TO_SOT_THT:TO-92_Inline, F.Cu at (245.1, 43.2)
- added encoder1: Conn_01x04_Female, Connector_PinSocket_2.54mm:PinSocket_1x04_P2.54mm_Horizontal, F.Cu at (236.5, 37.2)
- added laser_B1: Conn_01x02_Female, Connector_PinSocket_2.54mm:PinSocket_1x02_P2.54mm_Horizontal, F.Cu at (245.1, 37.2)
- added laser_G1: Conn_01x02_Female, Connector_PinSocket_2.54mm:PinSocket_1x02_P2.54mm_Horizontal, F.Cu at (252.8, 37.2)
- added laser_R1: Conn_01x02_Female, Connector_PinSocket_2.54mm:PinSocket_1x02_P2.54mm_Horizontal, F.Cu at (260.1, 37.4)
- J1, U1: moved to B.Cu
- Xgain1, Xoffset1, Ygain1, Yoffset1: moved to F.Cu
- moved J1 256.9 mm to (273.5, 32.3), turned to 180 degrees
- moved R5 253.5 mm to (276.4, 118.6), turned to 180 degrees
- moved R6 250.4 mm to (276.9, 100.1), turned to -90 degrees
- moved U1 241.8 mm to (261.4, 57.9), turned to -90 degrees
- moved U3 238.8 mm to (260.1, 101.6), turned to 0 degrees
- moved R4 235.9 mm to (256.8, 109.2), turned to 180 degrees
- moved Ygain1 234.1 mm to (257.6, 135.3)
- moved R1 225.5 mm to (261.6, 96.3), turned to 90 degrees
- moved Yoffset1 212.2 mm to (243.9, 135.3)
- moved Xgain1 207.9 mm to (217.0, 133.8)
- moved Xoffset1 202.7 mm to (200.4, 132.0)
- moved R11 199.9 mm to (238.0, 118.4), turned to 180 degrees
- moved R12 198.2 mm to (238.0, 100.3), turned to -90 degrees
- moved R9 191.9 mm to (217.2, 112.8)
- moved R7 183.4 mm to (217.4, 95.0), turned to 90 degrees
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Connections:
- J1 pad 11: unconnected-(J1-Pad11) -> Net-(J1-Pad11)
- J1 pad 12: unconnected-(J1-Pad12) -> Net-(LCD_backligh1-Pad2)
- J1 pad 13: Earth -> Net-(J1-Pad13)
- J1 pad 14: unconnected-(J1-Pad14) -> GND
- J1 pad 20: unconnected-(J1-Pad20) -> GND
- J1 pad 25: unconnected-(J1-Pad25) -> GND
- J1 pad 29: Net-(J1-Pad29) -> unconnected-(J1-Pad29)
- J1 pad 3: unconnected-(J1-Pad3) -> Net-(J1-Pad3)
- J1 pad 30: unconnected-(J1-Pad30) -> GND
- J1 pad 31: Net-(J1-Pad31) -> unconnected-(J1-Pad31)
- J1 pad 33: unconnected-(J1-Pad33) -> Net-(J1-Pad33)
- J1 pad 34: unconnected-(J1-Pad34) -> GND
- J1 pad 35: unconnected-(J1-Pad35) -> Net-(J1-Pad35)
- J1 pad 36: unconnected-(J1-Pad36) -> Net-(J1-Pad36)
- J1 pad 39: Earth -> GND
- J1 pad 5: unconnected-(J1-Pad5) -> Net-(J1-Pad5)
- J1 pad 6: Earth -> GND
- J1 pad 9: unconnected-(J1-Pad9) -> GND
- U1 pad 5: Earth -> GND
- U1 pad 7: Earth -> GND
- U2 pad 5: Earth -> GND
- U3 pad 5: Earth -> GND
- Vi1 pad 2: Earth -> GND
- Xoffset1 pad 3: Earth -> GND
- Yoffset1 pad 3: Earth -> GND
- galX1 pad 2: Earth -> GND
- galY1 pad 2: Earth -> GND
Routing:
- net Earth: track 151.6 -> 0.00 mm
- net +15V: track 99.3 -> 0.00 mm
- net Net-(J1-Pad15): track 79.4 -> 0.00 mm
- net Net-(R5-Pad2): track 74.3 -> 0.00 mm
- net Net-(R11-Pad2): track 61.1 -> 0.00 mm
- net Net-(U3-Pad3): track 61.1 -> 0.00 mm
- net -15V: track 56.2 -> 0.00 mm
- net Net-(U2-Pad3): track 54.1 -> 0.00 mm
- net Net-(R1-Pad1): track 45.5 -> 0.00 mm
- net Net-(R12-Pad1): track 39.4 -> 0.00 mm
- net Net-(R7-Pad1): track 37.1 -> 0.00 mm
- net Net-(R11-Pad1): track 33.7 -> 0.00 mm
- net Net-(R6-Pad1): track 24.8 -> 0.00 mm
- net Net-(R4-Pad2): track 24.5 -> 0.00 mm
- net +5V: track 21.7 -> 0.00 mm
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Other:
- board outline removed
- board text removed: "+"
- board text removed: "-"
- board text removed: "37 31 29"
- board text removed: "JLCJLCJLCJLC"
- board text removed: "Vi"
- board text removed: "X"
- board text removed: "Y"
- board text removed: "laser"
- board text removed: "swchs"

Commit message: RGB ildareader
Parts:
- removed LCD1: Conn_01x04_Female, Connector_PinSocket_2.54mm:PinSocket_1x04_P2.54mm_Horizontal
- removed LCD_backligh1: Conn_01x02_Female, Connector_PinSocket_2.54mm:PinSocket_1x02_P2.54mm_Horizontal
- added J2: Conn_01x05_Female, Connector_PinSocket_2.54mm:PinSocket_1x05_P2.54mm_Horizontal, B.Cu at (225.8, 34.8)
- encoder1, laser_B1, laser_G1, laser_R1: moved to B.Cu
- moved laser_B1 25.5 mm to (270.5, 34.9)
- moved Q2 13.3 mm to (273.1, 40.3)
- moved Q1 13.1 mm to (265.4, 40.1)
- moved Q3 13.1 mm to (257.8, 40.1)
- moved laser_G1 10.4 mm to (262.9, 34.9)
- moved J1 7.65 mm to (276.9, 25.4)
- moved laser_R1 5.48 mm to (255.3, 34.9)
- moved encoder1 5.27 mm to (241.3, 34.9)
Other:
- board text added: "B"
- board text added: "BTN"
- board text added: "G"
- board text added: "GND"
- board text added: "LASER"
- board text added: "LCD"
- board text added: "PWR"
- board text added: "R"
- board text added: "SCL"
- board text added: "SDA"
- board text added: "backlight"
- board text added: "enc_A"
- board text added: "enc_B"
- board text added: "encoder"

Commit message: pcb
Parts:
- added +15supply1: Conn_01x02_Male, Connector_PinHeader_2.54mm:PinHeader_1x02_P2.54mm_Horizontal, F.Cu at (112.9, 68.9)
- added -15debug1: Conn_01x01_Male, Connector_PinHeader_2.54mm:PinHeader_1x01_P2.54mm_Horizontal, F.Cu at (135.6, 56.4)
- added C1: 1u, Capacitor_THT:C_Disc_D5.0mm_W2.5mm_P5.00mm, F.Cu at (119.1, 38.2)
- added C2: 10u, Capacitor_THT:CP_Radial_Tantal_D5.5mm_P2.50mm, F.Cu at (119.9, 43.8)
- added C3: 10u, Capacitor_THT:CP_Radial_Tantal_D5.5mm_P2.50mm, F.Cu at (127.1, 43.8)
- added D1: D_Schottky, Diode_THT:D_A-405_P10.16mm_Horizontal, F.Cu at (134.9, 51.9)
- added D2: D, Diode_THT:D_A-405_P10.16mm_Horizontal, F.Cu at (112.2, 64.5)
- added R10: R, Resistor_THT:R_Axial_DIN0207_L6.3mm_D2.5mm_P10.16mm_Horizontal, F.Cu at (173.2, 35.7)
- added R13: 39k, Resistor_THT:R_Axial_DIN0207_L6.3mm_D2.5mm_P10.16mm_Horizontal, F.Cu at (160.8, 68.9)
- added R14: 2k2, Resistor_THT:R_Axial_DIN0207_L6.3mm_D2.5mm_P10.16mm_Horizontal, F.Cu at (160.8, 64.8)
- added R15: 47k, Resistor_THT:R_Axial_DIN0207_L6.3mm_D2.5mm_P10.16mm_Horizontal, F.Cu at (139.1, 60.7)
- added R2: R, Resistor_THT:R_Axial_DIN0207_L6.3mm_D2.5mm_P10.16mm_Horizontal, F.Cu at (169.2, 25.5)
- added R3: R, Resistor_THT:R_Axial_DIN0207_L6.3mm_D2.5mm_P10.16mm_Horizontal, F.Cu at (186.2, 30.6)
- added R8: R, Resistor_THT:R_Axial_DIN0207_L6.3mm_D2.5mm_P10.16mm_Horizontal, F.Cu at (186.2, 48.1)
- added U4: LM358, Package_DIP:DIP-8_W7.62mm, F.Cu at (178.5, 35.8)
- added U5: ADC0831, Package_DIP:DIP-8_W7.62mm, F.Cu at (191.6, 35.9)
- added U6: AOZ1282CI, Package_TO_SOT_SMD:SOT-23-6, F.Cu at (175.1, 65.0)
- added bat_probe1: Conn_01x01_Male, Connector_PinHeader_2.54mm:PinHeader_1x01_P2.54mm_Horizontal, F.Cu at (165.3, 35.7)
- added pwrSW1: Conn_01x03_Male, Connector_PinHeader_2.54mm:PinHeader_1x03_P2.54mm_Horizontal, F.Cu at (106.5, 38.5)
- added pwrSW_PU1: 47k, Resistor_THT:R_Axial_DIN0207_L6.3mm_D2.5mm_P10.16mm_Horizontal, F.Cu at (105.7, 47.9)
Connections:
- J1 pad 1: unconnected-(J1-Pad1) -> +3V3
- J1 pad 16: unconnected-(J1-Pad16) -> Net-(J1-Pad16)
- J1 pad 17: unconnected-(J1-Pad17) -> +3V3
- J1 pad 29: unconnected-(J1-Pad29) -> Net-(J1-Pad29)
- J1 pad 31: unconnected-(J1-Pad31) -> Net-(J1-Pad31)
- J1 pad 37: Net-(J1-Pad37) -> unconnected-(J1-Pad37)
- J1 pad 40: unconnected-(J1-Pad40) -> Net-(J1-Pad40)
- encoder1 pad 2: Net-(J1-Pad37) -> Net-(J1-Pad29)
- encoder1 pad 3: Net-(J1-Pad36) -> Net-(J1-Pad31)
- laser_B1 pad 2: Net-(laser_B1-Pad2) -> Net-(J1-Pad11)
- laser_G1 pad 2: Net-(laser_G1-Pad2) -> Net-(J1-Pad13)
- laser_R1 pad 2: Net-(laser_R1-Pad2) -> Net-(J1-Pad15)
Routing:
- net Net-(R10-Pad2): track 0.00 -> 29.7 mm
- net GND: track 0.00 -> 22.4 mm
- net Net-(R3-Pad2): track 0.00 -> 21.0 mm
- net +5V: track 0.00 -> 19.2 mm
- net Net-(R2-Pad1): track 0.00 -> 11.8 mm
- net Net-(R10-Pad1): track 0.00 -> 11.3 mm

Commit message: pcb done
Parts:
- added L1: 20u, Inductor_THT:L_Toroid_Vertical_L14.7mm_W8.6mm_P5.58mm_Pulse_KM-1, F.Cu at (95.7, 58.9)
- added L2: 20u, Inductor_THT:L_Toroid_Vertical_L14.7mm_W8.6mm_P5.58mm_Pulse_KM-1, F.Cu at (79.4, 58.9)
Changed lines of the file:
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@@
+    )
+  )
+  (footprint "Inductor_THT:L_Toroid_Vertical_L14.7mm_W8.6mm_P5.58mm_Pulse_KM-1" (layer "F.Cu")
+    (at 95.7 58.9)
+    (descr "L_Toroid, Vertical series, Radial, pin pitch=5.58mm, , length*width=14.73*8.64mm^2, Pulse, KM-1, http://datasheet.octopart.com/PE-92112KNL-Pulse-datasheet-17853305.pdf")
+    (tags "L_Toroid Vertical series Radial pin pitch 5.58mm  length 14.73mm width 8.64mm Pulse KM-1")
+    (property "Sheetfile" "pcb.kicad_sch")
+    (property "Sheetname" "")
+    (attr through_hole)
+    (fp_text reference "L1" (at 0 -3.05) (layer "F.SilkS")
+      (effects (font (size 1 1) (thickness 0.15)))
+    )
+    (fp_text value "20u" (at 0 8.63) (layer "F.Fab")
+      (effects (font (size 1 1) (thickness 0.15)))
+    )
+    (fp_text user "${REFERENCE}" (at 2.79 0) (layer "F.Fab")
+      (effects (font (size 1 1) (thickness 0.15)))
+    )
+    (fp_line (start 1.365 -1.65) (end 7.485 -1.65) (layer "F.SilkS") (width 0.12))
+    (fp_line (start -7.485 -1.65) (end -7.485 7.23) (layer "F.SilkS") (width 0.12))
+    (fp_line (start 7.485 -1.65) (end 7.485 7.23) (layer "F.SilkS") (width 0.12))
+    (fp_line (start -7.485 7.23) (end -1.365 7.23) (layer "F.SilkS") (width 0.12))
+    (fp_line (start 1.365 7.23) (end 7.485 7.23) (layer "F.SilkS") (width 0.12))
+    (fp_line (start -7.485 -1.65) (end -1.365 -1.65) (layer "F.SilkS") (width 0.12))
+    (fp_line (start 7.62 -2.05) (end -7.62 -2.05) (layer "F.CrtYd") (width 0.05))
+    (fp_line (start -7.62 -2.05) (end -7.62 7.63) (layer "F.CrtYd") (width 0.05))
+    (fp_line (start 7.62 7.63) (end 7.62 -2.05) (layer "F.CrtYd") (width 0.05))
+    (fp_line (start -7.62 7.63) (end 7.62 7.63) (layer "F.CrtYd") (width 0.05))
+    (fp_line (start -5.892 5.58) (end 5.892 5.58) (layer "F.Fab") (width 0.1))
+    (fp_line (start 4.7136 0) (end 5.3028 5.58) (layer "F.Fab") (width 0.1))
+    (fp_line (start 0 0) (end 0.5892 5.58) (layer "F.Fab") (width 0.1))
+    (fp_line (start 3.5352 0) (end 4.1244 5.58) (layer "F.Fab") (width 0.1))
+    (fp_line (start 2.3568 0) (end 2.946 5.58) (layer "F.Fab") (width 0.1))
+    (fp_line (start -3.5352 0) (end -2.946 5.58) (layer "F.Fab") (width 0.1))
+    (fp_line (start -4.7136 0) (end -4.1244 5.58) (layer "F.Fab") (width 0.1))
+    (fp_line (start -1.1784 0) (end -0.5892 5.58) (layer "F.Fab") (width 0.1))
+    (fp_line (start 1.1784 0) (end 1.7676 5.58) (layer "F.Fab") (width 0.1))
+    (fp_line (start -5.892 0) (end -5.892 5.58) (layer "F.Fab") (width 0.1))
+    (fp_line (start 5.892 0) (end -5.892 0) (layer "F.Fab") (width 0.1))
+    (fp_line (start 5.892 5.58) (end 5.892 0) (layer "F.Fab") (width 0.1))
+    (fp_line (start 7.365 -1.53) (end -7.365 -1.53) (layer "F.Fab") (width 0.1))
+    (fp_line (start -7.365 7.11) (end 7.365 7.11) (layer "F.Fab") (width 0.1))
+    (fp_line (start 7.365 7.11) (end 7.365 -1.53) (layer "F.Fab") (width 0.1))
+    (fp_line (start -5.892 0) (end -5.3028 5.58) (layer "F.Fab") (width 0.1))
+    (fp_line (start -2.3568 0) (end -1.7676 5.58) (layer "F.Fab") (width 0.1))
+    (fp_line (start -7.365 -1.53) (end -7.365 7.11) (layer "F.Fab") (width 0.1))
+    (pad "1" thru_hole circle (at 0 0) (size 3.6 3.6) (drill 1.8) (layers *.Cu *.Mask)
+      (net 59 "Net-(C1-Pad1)") (pinfunction "1") (pintype "passive"))
+    (pad "2" thru_hole circle (at 0 5.58) (size 3.6 3.6) (drill 1.8) (layers *.Cu *.Mask)
+      (net 2 "GND") (pinfunction "2") (pintype "passive"))
+    (model "${KICAD6_3DMODEL_DIR}/Inductor_THT.3dshapes/L_Toroid_Vertical_L14.7mm_W8.6mm_P5.58mm_Pulse_KM-1.wrl"
+      (offset (xyz 0 0 0))
+      (scale (xyz 1 1 1))
+      (rotate (xyz 0 0 0))
     )
   )
@@
       (offset (xyz 0 0 0))
       (scale (xyz 1 1 1))
+      (rotate (xyz 0 0 0))
+    )
+  )
+  (footprint "Inductor_THT:L_Toroid_Vertical_L14.7mm_W8.6mm_P5.58mm_Pulse_KM-1" (layer "F.Cu")
+    (at 79.41 58.9)
+    (descr "L_Toroid, Vertical series, Radial, pin pitch=5.58mm, , length*width=14.73*8.64mm^2, Pulse, KM-1, http://datasheet.octopart.com/PE-92112KNL-Pulse-datasheet-17853305.pdf")
+    (tags "L_Toroid Vertical series Radial pin pitch 5.58mm  length 14.73mm width 8.64mm Pulse KM-1")
+    (property "Sheetfile" "pcb.kicad_sch")
+    (property "Sheetname" "")
+    (attr through_hole)
+    (fp_text reference "L2" (at 0 -3.05) (layer "F.SilkS")
+      (effects (font (size 1 1) (thickness 0.15)))
+    )
+    (fp_text value "20u" (at 0 8.63) (layer "F.Fab")
+      (effects (font (size 1 1) (thickness 0.15)))
+    )
+    (fp_text user "${REFERENCE}" (at 2.79 0) (layer "F.Fab")
+      (effects (font (size 1 1) (thickness 0.15)))
+    )
+    (fp_line (start 1.365 7.23) (end 7.485 7.23) (layer "F.SilkS") (width 0.12))
+    (fp_line (start -7.485 -1.65) (end -1.365 -1.65) (layer "F.SilkS") (width 0.12))
+    (fp_line (start 7.485 -1.65) (end 7.485 7.23) (layer "F.SilkS") (width 0.12))
+    (fp_line (start -7.485 -1.65) (end -7.485 7.23) (layer "F.SilkS") (width 0.12))
+    (fp_line (start 1.365 -1.65) (end 7.485 -1.65) (layer "F.SilkS") (width 0.12))
+    (fp_line (start -7.485 7.23) (end -1.365 7.23) (layer "F.SilkS") (width 0.12))
+    (fp_line (start 7.62 7.63) (end 7.62 -2.05) (layer "F.CrtYd") (width 0.05))
+    (fp_line (start -7.62 7.63) (end 7.62 7.63) (layer "F.CrtYd") (width 0.05))
+    (fp_line (start -7.62 -2.05) (end -7.62 7.63) (layer "F.CrtYd") (width 0.05))
+    (fp_line (start 7.62 -2.05) (end -7.62 -2.05) (layer "F.CrtYd") (width 0.05))
+    (fp_line (start -7.365 -1.53) (end -7.365 7.11) (layer "F.Fab") (width 0.1))
+    (fp_line (start 5.892 0) (end -5.892 0) (layer "F.Fab") (width 0.1))
+    (fp_line (start -7.365 7.11) (end 7.365 7.11) (layer "F.Fab") (width 0.1))
+    (fp_line (start -2.3568 0) (end -1.7676 5.58) (layer "F.Fab") (width 0.1))
+    (fp_line (start 3.5352 0) (end 4.1244 5.58) (layer "F.Fab") (width 0.1))
+    (fp_line (start -5.892 0) (end -5.892 5.58) (layer "F.Fab") (width 0.1))
+    (fp_line (start -4.7136 0) (end -4.1244 5.58) (layer "F.Fab") (width 0.1))
+    (fp_line (start 2.3568 0) (end 2.946 5.58) (layer "F.Fab") (width 0.1))
+    (fp_line (start 7.365 -1.53) (end -7.365 -1.53) (layer "F.Fab") (width 0.1))
+    (fp_line (start 5.892 5.58) (end 5.892 0) (layer "F.Fab") (width 0.1))
+    (fp_line (start 1.1784 0) (end 1.7676 5.58) (layer "F.Fab") (width 0.1))
+    (fp_line (start -5.892 5.58) (end 5.892 5.58) (layer "F.Fab") (width 0.1))
+    (fp_line (start 4.7136 0) (end 5.3028 5.58) (layer "F.Fab") (width 0.1))
+    (fp_line (start -3.5352 0) (end -2.946 5.58) (layer "F.Fab") (width 0.1))
+    (fp_line (start -5.892 0) (end -5.3028 5.58) (layer "F.Fab") (width 0.1))
+    (fp_line (start -1.1784 0) (end -0.5892 5.58) (layer "F.Fab") (width 0.1))
+    (fp_line (start 0 0) (end 0.5892 5.58) (layer "F.Fab") (width 0.1))
+    (fp_line (start 7.365 7.11) (end 7.365 -1.53) (layer "F.Fab") (width 0.1))
+    (pad "1" thru_hole circle (at 0 0) (size 3.6 3.6) (drill 1.8) (layers *.Cu *.Mask)
+      (net 61 "Net-(C2-Pad2)") (pinfunction "1") (pintype "passive"))
+    (pad "2" thru_hole circle (at 0 5.58) (size 3.6 3.6) (drill 1.8) (layers *.Cu *.Mask)
+      (net 34 "-15V") (pinfunction "2") (pintype "passive"))
+    (model "${KICAD6_3DMODEL_DIR}/Inductor_THT.3dshapes/L_Toroid_Vertical_L14.7mm_W8.6mm_P5.58mm_Pulse_KM-1.wrl"
+      (offset (xyz 0 0 0))
+      (scale (xyz 1 1 1))

Commit message: pcb done
Parts:
- removed -15debug1: Conn_01x01_Male, Connector_PinHeader_2.54mm:PinHeader_1x01_P2.54mm_Horizontal
- removed J2: Conn_01x05_Female, Connector_PinSocket_2.54mm:PinSocket_1x05_P2.54mm_Horizontal
- removed Q1, Q2, Q3: BC547, Package_TO_SOT_THT:TO-92_Inline
- removed Vi1: Conn_01x03_Male, Connector_PinHeader_2.54mm:PinHeader_1x03_P2.54mm_Horizontal
- added LCD1: Conn_01x05_Male, Connector_PinHeader_2.54mm:PinHeader_1x05_P2.54mm_Horizontal, B.Cu at (238.4, 32.6)
- added galPWR1: Conn_01x03_Male, Connector_PinHeader_2.54mm:PinHeader_1x03_P2.54mm_Horizontal, B.Cu at (262.6, 73.6)
- +15supply1, C2, bat_probe1, galX1, galY1, pwrSW1: moved to B.Cu
- L1, L2: footprint Inductor_THT:L_Toroid_Vertical_L14.7mm_W8.6mm_P5.58mm_Pulse_KM-1 -> Inductor_SMD:L_Sumida_CR75; moved to B.Cu
- U1: moved to F.Cu
- encoder1: value Conn_01x04_Female -> Conn_01x04_Male; footprint Connector_PinSocket_2.54mm:PinSocket_1x04_P2.54mm_Horizontal -> Connector_PinHeader_2.54mm:PinHeader_1x04_P2.54mm_Horizontal
- laser_B1, laser_G1, laser_R1: value Conn_01x02_Female -> Conn_01x02_Male; footprint Connector_PinSocket_2.54mm:PinSocket_1x02_P2.54mm_Horizontal -> Connector_PinHeader_2.54mm:PinHeader_1x02_P2.54mm_Horizontal
- moved L2 192.0 mm to (271.4, 57.4), turned to -90 degrees
- moved L1 169.5 mm to (265.0, 67.1), turned to 90 degrees
- moved +15supply1 158.1 mm to (270.6, 80.3)
- moved C2 153.4 mm to (270.9, 71.2)
- moved C3 148.1 mm to (273.5, 65.6), turned to 180 degrees
- moved pwrSW_PU1 145.7 mm to (251.4, 48.2)
- moved pwrSW1 145.2 mm to (251.5, 32.6), turned to 90 degrees
- moved D2 143.9 mm to (256.1, 59.2)
- moved C1 129.4 mm to (248.1, 47.5), turned to -90 degrees
- moved D1 121.2 mm to (256.1, 55.3)
- moved R15 110.4 mm to (249.3, 66.8)
- moved Ygain1 103.7 mm to (227.5, 36.1), turned to 0 degrees
- moved R2 97.2 mm to (263.8, 48.2), turned to 0 degrees
- moved U6 96.7 mm to (271.6, 57.9)
- moved R13 93.2 mm to (253.5, 59.0), turned to 180 degrees
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Connections:
- J1 pad 1: +3V3 -> unconnected-(J1-Pad1)
- J1 pad 17: +3V3 -> unconnected-(J1-Pad17)
- encoder1 pad 1: GND -> Net-(J1-Pad33)
- encoder1 pad 2: Net-(J1-Pad29) -> Net-(J1-Pad31)
- encoder1 pad 3: Net-(J1-Pad31) -> Net-(J1-Pad29)
- encoder1 pad 4: Net-(J1-Pad33) -> GND
- laser_B1 pad 1: GND -> Net-(J1-Pad11)
- laser_B1 pad 2: Net-(J1-Pad11) -> GND
- laser_G1 pad 1: GND -> Net-(J1-Pad13)
- laser_G1 pad 2: Net-(J1-Pad13) -> GND
- laser_R1 pad 1: GND -> Net-(J1-Pad15)
- laser_R1 pad 2: Net-(J1-Pad15) -> GND
Routing:
- net GND: track 22.4 -> 245.9 mm
- net +5V: track 19.2 -> 136.9 mm
- net +15V: track 0.00 -> 93.7 mm
- net -15V: track 0.00 -> 85.9 mm
- net Net-(R5-Pad2): track 0.00 -> 71.0 mm, vias 0 -> 3
- net Net-(R11-Pad2): track 0.00 -> 56.9 mm
- net Net-(C1-Pad1): track 0.00 -> 56.0 mm
- net Net-(J1-Pad33): track 0.00 -> 55.6 mm
- net Net-(J1-Pad31): track 0.00 -> 54.9 mm
- net Net-(R4-Pad2): track 0.00 -> 52.9 mm, vias 0 -> 1
- net Net-(J1-Pad29): track 0.00 -> 52.2 mm
- net Net-(R5-Pad1): track 0.00 -> 52.1 mm
- net Net-(R1-Pad1): track 0.00 -> 50.8 mm
- net Net-(J1-Pad12): track 0.00 -> 48.2 mm
- net Net-(J1-Pad3): track 0.00 -> 45.5 mm
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Other:
- board outline added: 56.3 x 62.8 mm
- board text added: "+15V"
- board text added: "-15V"
- board text added: "15V"
- board text added: "5V"
- board text added: "GP23"
- board text added: "IN"
- board text added: "X+"
- board text added: "X-"
- board text added: "X0"
- board text added: "Y+"
- board text added: "Y-"
- board text added: "Y0"
- board text added: "bat %"
- board text added: "gh /phuid"
- board text added: "relay"

Commit message: pcb todo capacitors
Parts:
- removed G***: LOGO, LOGO
- moved R5 5.84 mm to (260.8, 75.9)
- moved R6 2.26 mm to (251.4, 76.8)
- moved +15supply1 1.32 mm to (271.4, 81.4)
- moved galPWR1 0.77 mm to (263.3, 73.5)
- moved galY1 0.48 mm to (253.4, 73.6)
Routing:
- net GND: track 245.9 -> 255.0 mm, vias 0 -> 1
- net +15V: track 93.7 -> 98.9 mm, vias 0 -> 1
- net Net-(R5-Pad1): track 52.1 -> 56.5 mm
- net Net-(R5-Pad2): track 71.0 -> 74.6 mm
- net Net-(J1-Pad29): track 52.2 -> 55.2 mm
- net Net-(J1-Pad33): track 55.6 -> 58.2 mm
- net Net-(J1-Pad31): track 54.9 -> 56.6 mm
- net Net-(R4-Pad2): track 52.9 -> 54.3 mm
- net Net-(R2-Pad1): track 43.5 -> 44.1 mm
Other:
- board text removed: "github.com/phuid"

Commit message: konzult pcb with tom
Parts:
- C2: footprint Capacitor_THT:CP_Radial_Tantal_D5.5mm_P2.50mm -> Capacitor_THT:CP_Radial_D5.0mm_P2.00mm
- Ce: renamed from C3; footprint Capacitor_THT:CP_Radial_Tantal_D5.5mm_P2.50mm -> Capacitor_THT:CP_Radial_D5.0mm_P2.00mm
- D1, D2: footprint Diode_THT:D_A-405_P10.16mm_Horizontal -> Diode_SMD:D_SMC_Handsoldering
- moved D2 10.4 mm to (264.7, 65.0), turned to 90 degrees
- moved D1 5.77 mm to (261.7, 56.7)
- moved L2 0.89 mm to (270.6, 57.4)
Routing:
- net -15V: track 86.3 -> 95.7 mm
- net Net-(U3-Pad3): track 26.5 -> 18.6 mm, vias 0 -> 1
- net Net-(R4-Pad2): track 54.3 -> 59.3 mm
- net Net-(R2-Pad1): track 44.1 -> 39.7 mm
- net Net-(C1-Pad2): track 24.1 -> 28.1 mm, vias 0 -> 1
- net Net-(C1-Pad1): track 56.3 -> 59.5 mm, vias 0 -> 3
- net Net-(R7-Pad2): track 0.00 -> 2.99 mm
- net Net-(R13-Pad2): track 31.7 -> 34.6 mm
- net GND: track 255.0 -> 257.6 mm
- net Net-(C2-Pad2): track 37.4 -> 34.8 mm, vias 0 -> 2
- net +15V: track 98.9 -> 100.6 mm
- net Net-(R15-Pad1): track 26.7 -> 27.5 mm
- net Net-(R10-Pad1): track 45.6 -> 46.3 mm
- net Net-(U2-Pad3): track 18.1 -> 17.4 mm, vias 0 -> 1
- net Net-(R3-Pad2): track 22.8 -> 22.6 mm, vias 0 -> 1
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Other:
- board text removed: "gh /phuid"
