File: pcb/kicad/pcb.kicad_pcb (KiCad board)
At the start: 2 copper layers, 56.3 x 62.8 mm, 45 parts, among them J1 Raspberry_Pi_2_3, U1 MCP4822, U2 TL082, U3 TL082, U4 LM358, U5 ADC0831, U6 AOZ1282CI

Commit message: PCB
Parts:
- moved U6 1.70 mm to (270.1, 59.4)
- moved R12 0.09 mm to (245.3, 65.6)
Routing:
- net Net-(C2-Pad2): track 32.1 -> 38.8 mm
- net Net-(R7-Pad1): track 22.2 -> 25.2 mm
- net Net-(R5-Pad1): track 11.6 -> 13.8 mm
- net Net-(R5-Pad2): track 63.7 -> 65.9 mm
- net Net-(R11-Pad2): track 38.7 -> 40.8 mm
- net Net-(R4-Pad2): track 6.04 -> 7.85 mm
- net Net-(R6-Pad1): track 23.2 -> 24.7 mm
- net Net-(C1-Pad2): track 26.6 -> 25.1 mm
- net Net-(R11-Pad1): track 10.6 -> 11.9 mm
- net Net-(R12-Pad1): track 9.52 -> 10.7 mm
- net -15V: track 56.7 -> 57.8 mm
- net Net-(R13-Pad2): track 11.6 -> 10.6 mm
- net +5V: track 100.6 -> 101.4 mm
- net +15V: track 108.9 -> 109.7 mm
- net Net-(R10-Pad1): track 16.8 -> 17.6 mm
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
Commit message: rpi power pcb
Routing:
- net +5V: track 101.4 -> 157.1 mm
Other:
- board text removed: "PWR"
Changed lines of the file:
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@@
     (effects (font (size 1 1) (thickness 0.15)))
   )
-  (gr_text "PWR" (at 230.6028 24.8366 -270) (layer "F.SilkS")
+  (gr_text "5V" (at 230.7844 24.5618 90) (layer "F.SilkS")
     (effects (font (size 1 1) (thickness 0.15)))
   )
@@
   (segment (start 278.13 52.07) (end 278.13 50.0888) (width 0.25) (layer "B.Cu") (net 16))
   (segment (start 251.901907 45.965511) (end 250.0884 44.152004) (width 0.25) (layer "B.Cu") (net 16))
+  (segment (start 264.414 38.3794) (end 265.176 39.1414) (width 0.25) (layer "F.Cu") (net 19))
   (segment (start 249.684311 35.994889) (end 261.074189 35.994889) (width 0.25) (layer "F.Cu") (net 19))
-  (segment (start 264.254789 38.534889) (end 265.176 39.4561) (width 0.25) (layer "F.Cu") (net 19))
+  (segment (start 261.074189 35.994889) (end 263.4587 38.3794) (width 0.25) (layer "F.Cu") (net 19))
+  (segment (start 263.4587 38.3794) (end 264.414 38.3794) (width 0.25) (layer "F.Cu") (net 19))
   (segment (start 248.3258 37.3534) (end 249.684311 35.994889) (width 0.25) (layer "F.Cu") (net 19))
-  (segment (start 265.176 39.4561) (end 265.176 43.561) (width 0.25) (layer "F.Cu") (net 19))
-  (segment (start 261.074189 35.994889) (end 263.614189 38.534889) (width 0.25) (layer "F.Cu") (net 19))
-  (segment (start 263.614189 38.534889) (end 264.254789 38.534889) (width 0.25) (layer "F.Cu") (net 19))
+  (segment (start 265.176 39.1414) (end 265.176 43.561) (width 0.25) (layer "F.Cu") (net 19))
   (via (at 265.176 43.561) (size 0.8) (drill 0.4) (layers "F.Cu" "B.Cu") (net 19))
   (segment (start 267.97 48.26) (end 276.86 48.26) (width 0.25) (layer "B.Cu") (net 19))
@@
   (segment (start 232.8774 38.227) (end 234.127 38.227) (width 0.25) (layer "B.Cu") (net 36))
   (segment (start 235 44.7032) (end 236.5502 46.2534) (width 0.25) (layer "B.Cu") (net 36))
-  (segment (start 277.6982 23.6982) (end 279.4 25.4) (width 0.5) (layer "F.Cu") (net 37))
+  (segment (start 274.1676 37.221) (end 274.1676 35.5386) (width 0.5) (layer "F.Cu") (net 37))
+  (segment (start 274.4062 23.6982) (end 278.6126 23.6982) (width 0.5) (layer "F.Cu") (net 37))
+  (segment (start 230.759 32.5882) (end 230.759 30.4038) (width 1) (layer "F.Cu") (net 37))
   (segment (start 251.37455 44.9734) (end 252.2982 44.04975) (width 0.5) (layer "F.Cu") (net 37))
-  (segment (start 274.1676 37.221) (end 274.1676 35.5386) (width 0.5) (layer "F.Cu") (net 37))
+  (segment (start 274.4062 35.3) (end 274.4062 23.6982) (width 0.5) (layer "F.Cu") (net 37))
   (segment (start 279.4 27.94) (end 279.4 25.4) (width 0.75) (layer "F.Cu") (net 37))
-  (segment (start 275.962778 23.6982) (end 277.6982 23.6982) (width 0.5) (layer "F.Cu") (net 37))
-  (segment (start 274.4062 35.3) (end 274.4062 25.254778) (width 0.5) (layer "F.Cu") (net 37))
-  (segment (start 274.4062 25.254778) (end 275.962778 23.6982) (width 0.5) (layer "F.Cu") (net 37))
   (segment (start 274.1676 35.5386) (end 274.4062 35.3) (width 0.5) (layer "F.Cu") (net 37))
+  (segment (start 230.759 30.4038) (end 237.8202 23.3426) (width 1) (layer "F.Cu") (net 37))
+  (segment (start 278.257 23.3426) (end 279.4 24.4856) (width 1) (layer "F.Cu") (net 37))
+  (segment (start 279.4 24.4856) (end 279.4 25.4) (width 1) (layer "F.Cu") (net 37))
+  (segment (start 278.6126 23.6982) (end 279.4 24.4856) (width 0.5) (layer "F.Cu") (net 37))
   (segment (start 248.3258 44.9734) (end 251.37455 44.9734) (width 0.5) (layer "F.Cu") (net 37))
   (segment (start 252.2982 44.04975) (end 252.2982 43.0936) (width 0.5) (layer "F.Cu") (net 37))
+  (segment (start 237.8202 23.3426) (end 278.257 23.3426) (width 1) (layer "F.Cu") (net 37))
   (segment (start 232.2354 34.0646) (end 230.759 32.5882) (width 0.5) (layer "B.Cu") (net 37))
   (segment (start 244.3 40.9476) (end 244.3 34.9) (width 0.5) (layer "B.Cu") (net 37))
