File: pcb/kicad/pcb.kicad_sch (KiCad schematic)
At the start: 45 parts, among them J1 Raspberry_Pi_2_3, U1 MCP4822, U2 TL082, U3 TL082, U4 LM358, U5 ADC0831, U6 AOZ1282CI

Commit message: how i found pc
Parts:
- added C4: 100u, Capacitor_THT:C_Disc_D5.0mm_W2.5mm_P5.00mm, symbol Device:C
- added D3: LED, symbol Device:LED
- added R16: 680R, Resistor_SMD:R_1812_4532Metric_Pad1.30x3.40mm_HandSolder, symbol Device:R
Connections:
- net +15V: now also C4.2
- net -15V: now also D3.1 (K)
- net GND: now also C4.1, R16.2
- new net: D3.2 (A), R16.1
Changed lines of the file:
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@@
   (junction (at 224.79 127.635) (diameter 0) (color 0 0 0 0)
   )
+  (junction (at 184.785 147.955) (diameter 0) (color 0 0 0 0)
+  )
   (junction (at 145.415 149.225) (diameter 0) (color 0 0 0 0)
   )
@@
   (junction (at 167.005 149.225) (diameter 0) (color 0 0 0 0)
   )
+  (junction (at 114.935 154.94) (diameter 0) (color 0 0 0 0)
+  )
   (junction (at 196.85 50.165) (diameter 0) (color 0 0 0 0)
   )
   (junction (at 61.595 157.48) (diameter 0) (color 0 0 0 0)
   )
+  (junction (at 117.475 158.75) (diameter 0) (color 0 0 0 0)
+  )
   (junction (at 156.21 46.355) (diameter 0) (color 0 0 0 0)
   )
@@
     (stroke (width 0) (type default))
   )
+  (wire (pts (xy 191.135 154.305) (xy 191.135 147.955))
+    (stroke (width 0) (type default))
+  )
   (wire (pts (xy 70.485 84.455) (xy 90.805 84.455))
     (stroke (width 0) (type default))
@@
     (stroke (width 0) (type default))
   )
-  (wire (pts (xy 184.785 135.89) (xy 184.785 154.305))
+  (wire (pts (xy 184.785 135.89) (xy 184.785 147.955))
     (stroke (width 0) (type default))
   )
@@
     (stroke (width 0) (type default))
   )
+  (wire (pts (xy 120.015 158.75) (xy 117.475 158.75))
+    (stroke (width 0) (type default))
+  )
   (wire (pts (xy 114.935 133.35) (xy 114.935 149.86))
     (stroke (width 0) (type default))
@@
     (stroke (width 0) (type default))
   )
+  (wire (pts (xy 184.785 147.955) (xy 184.785 154.305))
+    (stroke (width 0) (type default))
+  )
   (wire (pts (xy 70.485 153.67) (xy 65.405 153.67))
     (stroke (width 0) (type default))
@@
     (stroke (width 0) (type default))
   )
+  (wire (pts (xy 120.015 175.26) (xy 120.015 158.75))
+    (stroke (width 0) (type default))
+  )
   (wire (pts (xy 224.79 127.635) (xy 224.79 133.985))
     (stroke (width 0) (type default))
@@
     (stroke (width 0) (type default))
   )
+  (wire (pts (xy 182.245 161.925) (xy 183.515 161.925))
+    (stroke (width 0) (type default))
+  )
   (wire (pts (xy 240.03 55.245) (xy 240.03 64.135))
     (stroke (width 0) (type default))
@@
     (stroke (width 0) (type default))
   )
+  (wire (pts (xy 182.245 149.225) (xy 174.625 149.225))
+    (stroke (width 0) (type default))
+  )
   (wire (pts (xy 207.01 75.565) (xy 203.2 75.565))
     (stroke (width 0) (type default))
@@
     (stroke (width 0) (type default))
   )
+  (wire (pts (xy 109.855 175.26) (xy 109.855 154.94))
+    (stroke (width 0) (type default))
+  )
+  (wire (pts (xy 114.935 154.94) (xy 114.935 158.75))
+    (stroke (width 0) (type default))
+  )
   (wire (pts (xy 47.625 90.805) (xy 110.49 90.805))
     (stroke (width 0) (type default))
@@
     (stroke (width 0) (type default))
   )
+  (wire (pts (xy 109.855 154.94) (xy 114.935 154.94))
+    (stroke (width 0) (type default))
+  )
+  (wire (pts (xy 191.135 147.955) (xy 184.785 147.955))
+    (stroke (width 0) (type default))
+  )
   (wire (pts (xy 61.595 172.72) (xy 61.595 157.48))
     (stroke (width 0) (type default))
@@
     (stroke (width 0) (type default))
   )
+  (wire (pts (xy 182.245 161.925) (xy 182.245 149.225))
+    (stroke (width 0) (type default))
+  )
   (wire (pts (xy 42.545 154.94) (xy 42.545 153.035))
     (stroke (width 0) (type default))
@@
     (stroke (width 0) (type default))
   )
-  (wire (pts (xy 114.935 149.86) (xy 114.935 158.75))
+  (wire (pts (xy 114.935 149.86) (xy 114.935 154.94))
     (stroke (width 0) (type default))
   )
@@
   )
   (wire (pts (xy 90.805 74.295) (xy 86.36 74.295))
+    (stroke (width 0) (type default))
+  )
+  (wire (pts (xy 112.395 175.26) (xy 109.855 175.26))
     (stroke (width 0) (type default))
   )
@@
     )
   )
+  (symbol (lib_id "Device:R") (at 191.135 158.115 180) (unit 1)
+    (in_bom yes) (on_board yes) (dnp no)
+    (property "Reference" "R16" (at 196.3928 158.115 90)
+      (effects (font (size 1.27 1.27)))
+    )
+    (property "Value" "680R" (at 194.0814 158.115 90)
+      (effects (font (size 1.27 1.27)))
+    )
+    (property "Footprint" "Resistor_SMD:R_1812_4532Metric_Pad1.30x3.40mm_HandSolder" (at 192.913 158.115 90)
+      (effects (font (size 1.27 1.27)) hide)
+    )
+    (property "Datasheet" "~" (at 191.135 158.115 0)
+      (effects (font (size 1.27 1.27)) hide)
+    )
+    (pin "1")
+    (pin "2")
+    (instances
+      (project "pcb"
+        (path "/407682a6-e2e1-4fd1-bd62-7d4bad485dba"
+          (reference "R16") (unit 1)
+        )
+      )
+    )
+  )
   (symbol (lib_id "power:GND") (at 47.625 113.665 90) (unit 1)
     (in_bom yes) (on_board yes) (dnp no) (fields_autoplaced)
@@
     )
   )
+  (symbol (lib_id "Device:LED") (at 187.325 161.925 0) (unit 1)
+    (in_bom yes) (on_board yes) (dnp no) (fields_autoplaced)
+    (property "Reference" "D3" (at 185.7375 156.5107 0)
+      (effects (font (size 1.27 1.27)))
+    )
+    (property "Value" "LED" (at 185.7375 158.9349 0)
+      (effects (font (size 1.27 1.27)))
+    )
+    (property "Footprint" "" (at 187.325 161.925 0)
+      (effects (font (size 1.27 1.27)) hide)
+    )
+    (property "Datasheet" "~" (at 187.325 161.925 0)
+      (effects (font (size 1.27 1.27)) hide)
+    )
+    (pin "2")
+    (pin "1")
+    (instances
+      (project "pcb"
+        (path "/407682a6-e2e1-4fd1-bd62-7d4bad485dba"
+          (reference "D3") (unit 1)
+        )
+      )
+    )
+  )
   (symbol (lib_id "Regulator_Switching:AOZ1282CI") (at 127.635 135.89 0) (unit 1)
     (in_bom yes) (on_board yes) (dnp no) (fields_autoplaced)
@@
         )
       )
+    )
+  )
+  (symbol (lib_id "Device:C") (at 116.205 175.26 270) (unit 1)
+    (in_bom yes) (on_board yes) (dnp no) (fields_autoplaced)
+    (property "Reference" "C4" (at 116.205 168.9567 90)
+      (effects (font (size 1.27 1.27)))
+    )
+    (property "Value" "100u" (at 116.205 171.3809 90)
+      (effects (font (size 1.27 1.27)))
+    )
+    (property "Footprint" "Capacitor_THT:C_Disc_D5.0mm_W2.5mm_P5.00mm" (at 112.395 176.2252 0)
+      (effects (font (size 1.27 1.27)) hide)
+    )
+    (property "Datasheet" "~" (at 116.205 175.26 0)
+      (effects (font (size 1.27 1.27)) hide)
+    )
+    (pin "1")
+    (pin "2")
+    (instances
+      (project "pcb"
+        (path "/407682a6-e2e1-4fd1-bd62-7d4bad485dba"
+          (reference "C4") (unit 1)
+        )
+      )
